Commit message: add file

File: Field.urdf (robot description, URDF)
Before this commit: robot plane, 1 links, 0 joints
Links:
- link field: geometry collision box size=200.0 200.0 0.1; visual box size=200.0 200.0 -0.1

File: box.urdf (robot description, URDF)
Before this commit: robot plane, 1 links, 0 joints
Links:
- added link cylinder, mass 1; collision cylinder length=0.05 radius=0.2; visual cylinder length=0.05 radius=0.2
- link box: mass None -> 1; geometry collision cylinder length=0.05 radius=0.2; visual cylinder length=0.05 radius=0.2
Joints:
- added joint world_to_box: type continuous, parent cylinder, child box, origin xyz=0 0 3 rpy=0 1.5707 0, axis 0 0 1, limit effort=0 velocity=0

Commit message: add file

File: Field.urdf (robot description, URDF)
Before this commit: robot plane, 1 links, 0 joints
Links:
- link field: geometry collision box size=200.0 200.0 0.1; visual box size=20.0 20.0 -0.1

Commit message: add file

File: Field.urdf (robot description, URDF)
Before this commit: robot plane, 1 links, 0 joints
Links:
- link field: geometry collision box size=200.0 200.0 0.1; visual box size=8.0 8.0 -0.1

Commit message: add file

File: Field.urdf (robot description, URDF)
Before this commit: robot plane, 1 links, 0 joints
Links:
- link field: geometry collision box size=8.0 8.0 -0.1; visual box size=8.0 8.0 0

Commit message: add file

File: Field.urdf (robot description, URDF)
Before this commit: robot plane, 1 links, 0 joints
Links:
- link field: geometry collision box size=4.0 4.0 -0.1; visual box size=4.0 4.0 0

Commit message: add file

File: Field.urdf (robot description, URDF)
Before this commit: robot plane, 1 links, 0 joints
Links:
- link field: geometry collision box size=4.0 4.0 0; visual box size=4.0 4.0 0

File: box.urdf (robot description, URDF)
Before this commit: robot plane, 2 links, 1 joints
Links:
- removed link box
- removed link cylinder
- added link corpus, mass 1; collision box size=0.1 0.1 0.2; visual box size=.2 .2 .2
Joints:
- removed joint world_to_box
