Commit message: add file

File: robot.urdf (robot description, URDF)
Before this commit: robot 2wheeledRobot, 4 links, 3 joints
Links:
- link center_wheel: geometry collision sphere radius=0.03; visual sphere radius=0.03
Joints:
- joint corpus_to_center_wheel: axis 0 0 1 -> 1 1 1; origin xyz=0.1 0 0 rpy=0 -1.5707 -1.5707 -> xyz=0.1 0 -0.03 rpy=0 0 0; type revolute -> spherical
- joint corpus_to_left_wheel: child left_wheel -> right_wheel; origin xyz=-0.1 -0.125 0 rpy=0 -1.5707 -1.5707 -> xyz=-0.1 0.125 0 rpy=0 -1.5707 -1.5707
- joint corpus_to_right_wheel: child right_wheel -> left_wheel; origin xyz=-0.1 0.125 0 rpy=0 -1.5707 -1.5707 -> xyz=-0.1 -0.125 0 rpy=0 -1.5707 -1.5707
